File: Placa_IoT/MCU_wifi_ble.kicad_sch (KiCad schematic)
At the start: 0 parts

Commit message: MCU en proceso
Parts:
- added C10, C11, C14, C7: 100 nf, Capacitor_SMD:C_0402_1005Metric, symbol Device:C
- added C12, C13: 12 pF, Capacitor_SMD:C_0402_1005Metric, symbol Device:C
- added C15, C16, C18, C20: NC, Capacitor_SMD:C_0402_1005Metric, symbol Device:C
- added C17, C19, C5, C9: 1 uf, Capacitor_SMD:C_0402_1005Metric, symbol Device:C
- added C6: 10 nf, Capacitor_SMD:C_0402_1005Metric, symbol Device:C
- added C8: 10 uf, Capacitor_SMD:C_0402_1005Metric, symbol Device:C
- added L1: 2 nH, Inductor_SMD:L_0402_1005Metric, symbol Device:L
- added L2: 22 nH, Inductor_SMD:L_0402_1005Metric, symbol Device:L
- added R4: NC, Resistor_SMD:R_0402_1005Metric, symbol Device:R
- added R5: 499 Ohm, Resistor_SMD:R_0402_1005Metric, symbol Device:R
- added U3: ESP32-S3, ic_control:QFN-56-1EP_7x7mm_P0.4mm_EP4x4mm, symbol IC_control:ESP32-S3
- added U4: PRO-OB-536, antennas:ANTENNA_PIFA_3D_2.4GHZ, symbol Antennas:ANTENNA_PIFA_3D_2.4GHZ
- added Y1: 40 mHz, Crystal:Crystal_SMD_3225-4Pin_3.2x2.5mm, symbol Device:Crystal_GND24
Connections:
- new net: C12.1, L2.1, Y1.1
- new net: L2.2, U3.54 (XTAL_P)
- new net: C11.1, L1.2, U3.2 (VDD3P3), U3.3 (VDD3P3)
- new net: R5.2, U3.49 (U0TXD)
- new net: C15.1, C17.1, U3.1 (LNA_IN)
- new net: C16.1, C17.2, C18.1, C19.1
- new net: C13.1, U3.53 (XTAL_N), Y1.3
- new net: C19.2, C20.1, U4.2 (FEED)
- new net +3.3V: C10.1, C14.1, C5.1, C6.1, C7.1, C8.1, C9.1, L1.1, R4.2, U3.20 (VDD3P3_RTC), U3.46 (VDD3P3_CPU), U3.55 (VDDA), U3.56 (VDDA)
- new net GND: C10.2, C11.2, C12.2, C13.2, C14.2, C15.2, C16.2, C18.2, C20.2, C5.2, C6.2, C7.2, C8.2, C9.2, U3.57 (GND), U4.1 (GND), Y1.2 (G), Y1.4 (G)
- new net IO0: U3.5 (GPIO0)
- new net IO1: U3.6 (GPIO1)
- new net IO3: U3.8 (GPIO3)
- new net IO4: U3.9 (GPIO4)
- new net IO45: R4.1, U3.51 (GPIO45)
- new net IO5: U3.10 (GPIO5)
- new net IO6: U3.11 (GPIO6)
- new net IO7: U3.12 (GPIO7)
- new net IO8: U3.13 (GPIO8)
- new net IO9: U3.14 (GPIO9)
- new net RST/EN: U3.4 (CHIP_PU)
- new net SD0-MISO-IO2: U3.7 (GPIO2)
- no-connect marks 0 -> 7

Commit message: MCU en proceso 2
Connections:
- net IO3: now also U3.18 (GPIO13)
- net IO4: now also U3.19 (GPIO14)
- net IO5: now also U3.23 (GPIO17)
- net IO6: now also U3.24 (GPIO18)
- net IO7: now also U3.25 (GPIO19/USB_D-)
- net IO8: now also U3.26 (GPIO20/USB_D+)
- net IO9: now also U3.27 (GPIO21)
- net LORA_TX: now reaches U3.15 (GPIO10)
- net CMD-M0S1-IO11: now reaches U3.16 (GPIO11)
- net IO12: now reaches U3.17 (GPIO12)
Changed lines of the file:
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@@
+	(wire
+		(pts
+			(xy 88.9 118.11) (xy 106.68 118.11)
+		)
+		(stroke
+			(width 0)
+			(type default)
+		)
+	)
 	(wire
 		(pts
@@
 	(wire
 		(pts
+			(xy 88.9 123.19) (xy 106.68 123.19)
+		)
+		(stroke
+			(width 0)
+			(type default)
+		)
+	)
+	(wire
+		(pts
 			(xy 68.58 153.67) (xy 77.47 153.67)
 		)
@@
 	(wire
 		(pts
+			(xy 88.9 113.03) (xy 106.68 113.03)
+		)
+		(stroke
+			(width 0)
+			(type default)
+		)
+	)
+	(wire
+		(pts
 			(xy 106.68 138.43) (xy 93.98 138.43)
 		)
@@
 	(wire
 		(pts
+			(xy 88.9 102.87) (xy 106.68 102.87)
+		)
+		(stroke
+			(width 0)
+			(type default)
+		)
+	)
+	(wire
+		(pts
 			(xy 186.69 138.43) (xy 191.77 138.43)
 		)
@@
 	(wire
 		(pts
+			(xy 88.9 115.57) (xy 106.68 115.57)
+		)
+		(stroke
+			(width 0)
+			(type default)
+		)
+	)
+	(wire
+		(pts
 			(xy 207.01 138.43) (xy 210.82 138.43)
 		)
@@
 	(wire
 		(pts
+			(xy 88.9 105.41) (xy 106.68 105.41)
+		)
+		(stroke
+			(width 0)
+			(type default)
+		)
+	)
+	(wire
+		(pts
 			(xy 88.9 85.09) (xy 106.68 85.09)
 		)
@@
 	(wire
 		(pts
+			(xy 88.9 107.95) (xy 106.68 107.95)
+		)
+		(stroke
+			(width 0)
+			(type default)
+		)
+	)
+	(wire
+		(pts
 			(xy 119.38 50.8) (xy 119.38 69.85)
 		)
@@
 	(wire
 		(pts
+			(xy 88.9 125.73) (xy 106.68 125.73)
+		)
+		(stroke
+			(width 0)
+			(type default)
+		)
+	)
+	(wire
+		(pts
 			(xy 68.58 135.89) (xy 106.68 135.89)
 		)
@@
 	(wire
 		(pts
+			(xy 88.9 120.65) (xy 106.68 120.65)
+		)
+		(stroke
+			(width 0)
+			(type default)
+		)
+	)
+	(wire
+		(pts
 			(xy 127 69.85) (xy 127 26.67)
+		)
+		(stroke
+			(width 0)
+			(type default)
+		)
+	)
+	(wire
+		(pts
+			(xy 88.9 110.49) (xy 106.68 110.49)
 		)
 		(stroke
@@
 		)
 	)
+	(label "IO12"
+		(at 88.9 107.95 0)
+		(effects
+			(font
+				(size 1.27 1.27)
+			)
+			(justify left bottom)
+		)
+	)
 	(label "IO6"
 		(at 88.9 92.71 0)
@@
 		)
 	)
+	(label "IO7"
+		(at 88.9 120.65 0)
+		(effects
+			(font
+				(size 1.27 1.27)
+			)
+			(justify left bottom)
+		)
+	)
+	(label "CMD-M0S1-IO11"
+		(at 88.9 105.41 0)
+		(effects
+			(font
+				(size 1.27 1.27)
+			)
+			(justify left bottom)
+		)
+	)
+	(label "IO6"
+		(at 88.9 118.11 0)
+		(effects
+			(font
+				(size 1.27 1.27)
+			)
+			(justify left bottom)
+		)
+	)
 	(label "IO4"
 		(at 88.9 87.63 0)
@@
 		)
 	)
+	(label "IO5"
+		(at 88.9 115.57 0)
+		(effects
+			(font
+				(size 1.27 1.27)
+			)
+			(justify left bottom)
+		)
+	)
+	(label "IO9"
+		(at 88.9 125.73 0)
+		(effects
+			(font
+				(size 1.27 1.27)
+			)
+			(justify left bottom)
+		)
+	)
 	(label "IO0"
 		(at 88.9 77.47 0)
@@
 	)
 	(label "IO8"
+		(at 88.9 123.19 0)
+		(effects
+			(font
+				(size 1.27 1.27)
+			)
+			(justify left bottom)
+		)
+	)
+	(label "LORA_TX"
+		(at 88.9 102.87 0)
+		(effects
+			(font
+				(size 1.27 1.27)
+			)
+			(justify left bottom)
+		)
+	)
+	(label "IO8"
 		(at 88.9 97.79 0)
 		(effects
@@
 		(effects
 			(font
+				(size 1.27 1.27)
+			)
+			(justify left bottom)
+		)
+	)
+	(label "IO3"
+		(at 88.9 110.49 0)
+		(effects
+			(font
+				(size 1.27 1.27)
+			)
+			(justify left bottom)
+		)
+	)
+	(label "IO4"
+		(at 88.9 113.03 0)
+		(effects
+			(font

Commit message: MCU sin terminar
Parts:
- added J1, J2: 22-28-4144, connectors:CONN_THT_MV_PH_P2.54MM_P14, symbol Connectors:CONN_THT_MV_PH_P2.54MM_P14
- C15, C16, C18, C20, R4: now not fitted
Connections:
- net GND: now also J1.2 (Pin_2), J1.4 (Pin_4)
- net IO3: no longer U3.18 (GPIO13)
- net IO4: no longer U3.19 (GPIO14)
- net IO45: now also J1.13 (Pin_13), J1.7 (Pin_7)
- net IO5: no longer U3.23 (GPIO17)
- net IO6: no longer U3.24 (GPIO18)
- net IO7: no longer U3.25 (GPIO19/USB_D-)
- net IO8: no longer U3.26 (GPIO20/USB_D+)
- net IO9: no longer U3.27 (GPIO21)
- net UORTXD: now reaches R5.1
- net UORTXD: now also J1.12 (Pin_12)
- net IO15: now reaches U3.21 (XTAL_32K_P)
- net IO16: now reaches U3.22 (XTAL_32K_N)
- net IO48: now reaches U3.36 (SPICLK_N)
- net IO47: now reaches U3.37 (SPICLK_P)
- net IO33: now reaches U3.38 (GPIO33)
- net IO34: now reaches U3.39 (GPIO34)
- net IO35: now reaches U3.40 (GPIO35)
- net IO36: now reaches U3.41 (GPIO36)
- net IO37: now reaches U3.42 (GPIO37)
- net IO38: now reaches U3.43 (GPIO38)
- net IO39/MTCK: now reaches U3.44 (MTCK)
- net IO39/MTCK: now also J1.10 (Pin_10)
- net IO40/MTDO: now reaches U3.45 (MTDO)
- net IO40/MTDO: now also J1.9 (Pin_9)
- net IO41/MTDI: now reaches U3.47 (MTDI)
- net IO41/MTDI: now also J1.8 (Pin_8)
- net IO42/MTMS: now reaches U3.48 (MTMS)
- net IO42/MTMS: now also J1.5 (Pin_5)
- net UORDXD: now reaches U3.50 (U0RXD)
- net UORDXD: now also J1.11 (Pin_11)
- net IO46: now reaches U3.52 (GPIO46)
- net IO46: now also J1.6 (Pin_6)
- new net +3.3VP: J1.3 (Pin_3)
- new net CLK-SCK-IO14: U3.19 (GPIO14)
- new net DM: U3.25 (GPIO19/USB_D-)
- new net DP: U3.26 (GPIO20/USB_D+)
- new net IO17: U3.23 (GPIO17)
- new net IO18: U3.24 (GPIO18)
- new net LORA_RX: U3.27 (GPIO21)
- new net SD3-CS-IO13: U3.18 (GPIO13)
- new net VBAT: J1.14 (Pin_14)
- new net VBUS: J1.1 (Pin_1)
Other:
- moved on the sheet: C17, C19, R5, U4
