File: Placa_IoT/RF_LORA.kicad_sch (KiCad schematic)
At the start: 0 parts

Commit message: RF_LORA Iniciada
Parts:
- added U5: T-SX1262, ic_control:MODULE_T_SX1262, symbol IC_control:T_SX1262
Connections:
- new net GND: U5.1 (GND), U5.8 (GND)
- new net IO36: U5.2 (MISO), U5.6 (NRESET)
- new net IO5: U5.5 (NSS)
- new net IO7: U5.4 (SCK)
- new net IO8: U5.3 (MOSI)
